File: kicad/spiky_sphere.kicad_pcb (KiCad board)
At the start: 2 copper layers, 101.6 x 66 mm, 139 parts, among them K1 CONN_3, K2 CONN_3, K3 CONN_3, K4 CONN_3, K5 CONN_3, K6 CONN_3, K7 CONN_3, P1 CONN_8, U1 LED_MTX_5X7

Commit message: revised files... drill file glitch?
Other:
- net class Default: via_dia 1.016 -> 0.762; via_drill 0.635 -> 0.381
- rule via_min_drill: 0.508 -> 0.381
- rule via_min_size: 0.889 -> 0.762
Changed lines of the file:
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@@
     (segment_width 0.2)
     (edge_width 0.1)
-    (via_size 1.016)
-    (via_drill 0.635)
-    (via_min_size 0.889)
-    (via_min_drill 0.508)
+    (via_size 0.762)
+    (via_drill 0.381)
+    (via_min_size 0.762)
+    (via_min_drill 0.381)
     (uvia_size 0.508)
     (uvia_drill 0.127)
@@
     (clearance 0.254)
     (trace_width 0.254)
-    (via_dia 1.016)
-    (via_drill 0.635)
+    (via_dia 0.762)
+    (via_drill 0.381)
     (uvia_dia 0.508)
     (uvia_drill 0.127)
@@
   (segment (start 115.57 108.204) (end 119.126 108.204) (width 0.254) (layer B.Cu) (net 20))
   (segment (start 112.051 108.204) (end 115.57 108.204) (width 0.254) (layer B.Cu) (net 20))
-  (via (at 112.051 108.204) (size 1.016) (layers F.Cu B.Cu) (net 20))
+  (via (at 112.051 108.204) (size 0.762) (layers F.Cu B.Cu) (net 20))
   (segment (start 126.275 108.204) (end 126.238 108.204) (width 0.254) (layer B.Cu) (net 20))
-  (via (at 126.275 108.204) (size 1.016) (layers F.Cu B.Cu) (net 20))
+  (via (at 126.275 108.204) (size 0.762) (layers F.Cu B.Cu) (net 20))
   (segment (start 122.719 108.204) (end 122.682 108.204) (width 0.254) (layer B.Cu) (net 20))
-  (via (at 122.719 108.204) (size 1.016) (layers F.Cu B.Cu) (net 20))
+  (via (at 122.719 108.204) (size 0.762) (layers F.Cu B.Cu) (net 20))
   (segment (start 119.163 108.204) (end 119.126 108.204) (width 0.254) (layer B.Cu) (net 20))
-  (via (at 119.163 108.204) (size 1.016) (layers F.Cu B.Cu) (net 20))
+  (via (at 119.163 108.204) (size 0.762) (layers F.Cu B.Cu) (net 20))
   (segment (start 115.607 108.204) (end 115.57 108.204) (width 0.254) (layer B.Cu) (net 20))
-  (via (at 115.607 108.204) (size 1.016) (layers F.Cu B.Cu) (net 20))
+  (via (at 115.607 108.204) (size 0.762) (layers F.Cu B.Cu) (net 20))
   (segment (start 113.104 103.886) (end 116.078 103.886) (width 0.254) (layer F.Cu) (net 20))
   (segment (start 112.051 104.939) (end 113.104 103.886) (width 0.254) (layer F.Cu) (net 20))
@@
   (segment (start 91.223 104.939) (end 92.276 103.886) (width 0.254) (layer F.Cu) (net 20))
   (segment (start 92.276 103.886) (end 95.25 103.886) (width 0.254) (layer F.Cu) (net 20))
-  (via (at 94.779 108.204) (size 1.016) (layers F.Cu B.Cu) (net 20))
+  (via (at 94.779 108.204) (size 0.762) (layers F.Cu B.Cu) (net 20))
   (segment (start 94.779 108.204) (end 94.742 108.204) (width 0.254) (layer B.Cu) (net 20))
-  (via (at 98.335 108.204) (size 1.016) (layers F.Cu B.Cu) (net 20))
+  (via (at 98.335 108.204) (size 0.762) (layers F.Cu B.Cu) (net 20))
   (segment (start 98.335 108.204) (end 98.298 108.204) (width 0.254) (layer B.Cu) (net 20))
-  (via (at 101.891 108.204) (size 1.016) (layers F.Cu B.Cu) (net 20))
+  (via (at 101.891 108.204) (size 0.762) (layers F.Cu B.Cu) (net 20))
   (segment (start 101.891 108.204) (end 101.854 108.204) (width 0.254) (layer B.Cu) (net 20))
-  (via (at 105.447 108.204) (size 1.016) (layers F.Cu B.Cu) (net 20))
+  (via (at 105.447 108.204) (size 0.762) (layers F.Cu B.Cu) (net 20))
   (segment (start 105.447 108.204) (end 105.41 108.204) (width 0.254) (layer B.Cu) (net 20))
-  (via (at 91.223 108.204) (size 1.016) (layers F.Cu B.Cu) (net 20))
+  (via (at 91.223 108.204) (size 0.762) (layers F.Cu B.Cu) (net 20))
   (segment (start 91.223 108.204) (end 94.742 108.204) (width 0.254) (layer B.Cu) (net 20))
   (segment (start 94.742 108.204) (end 98.298 108.204) (width 0.254) (layer B.Cu) (net 20))

Commit message: small changes and added illum boards
Parts:
- removed the D16 at (182.6, 102.6)
- removed the D16 at (168.7, 102.6)
- removed the D17 at (182.6, 102.6)
- removed the D17 at (168.7, 102.6)
- removed the D18 at (182.6, 102.6)
- removed the D18 at (168.7, 102.6)
- removed the K6 at (182.6, 104.6)
- removed the K6 at (168.7, 104.6)
- removed the R6 at (182.6, 99.3)
- removed the R6 at (168.7, 99.3)
- added D22: XP-E2_LED, LED_LUW_CN5M, B.Cu at (168.7, 102.6)
- added D22: XP-E2_LED, LED_LUW_CN5M, B.Cu at (182.6, 102.6)
- added K8: CONN_3, CONN_3X1_MALE_SMT, F.Cu at (168.7, 102.6)
- added K8: CONN_3, CONN_3X1_MALE_SMT, F.Cu at (182.6, 102.6)
Connections:
- D10 pad 2: N-0000031 -> N-0000033
- D11 pad 2: N-0000031 -> N-0000033
- D12 pad 2: N-0000031 -> N-0000033
- D4 pad 2: N-0000029 -> N-0000031
- D5 pad 2: N-0000029 -> N-0000031
- D6 pad 2: N-0000029 -> N-0000031
- JP1 pad 1: N-0000015 -> N-000002
- JP1 pad 2: N-0000020 -> N-0000024
- JP2 pad 1: N-0000015 -> N-000002
- JP2 pad 2: N-0000018 -> N-0000023
- JP3 pad 1: N-0000015 -> N-000002
- JP3 pad 2: N-0000017 -> N-0000021
- JP4 pad 1: N-0000015 -> N-000002
- JP4 pad 2: N-0000016 -> N-0000014
- JP5 pad 1: N-0000015 -> N-000002
- JP5 pad 2: N-0000019 -> N-0000017
- P1 pad 1: N-000002 -> N-000005
- P1 pad 2: N-0000014 -> N-0000015
- P1 pad 3: N-0000013 -> N-0000016
- P1 pad 4: N-0000012 -> N-0000022
- P1 pad 5: N-0000011 -> N-0000018
- P1 pad 6: N-0000010 -> N-000004
- P1 pad 7: N-000009 -> N-000003
- P1 pad 8: N-0000015 -> N-000002
- R2 pad 1: N-0000029 -> N-0000031
- R4 pad 1: N-0000031 -> N-0000033
- U1 pad 1: N-0000018 -> N-0000023
- U1 pad 10: N-0000013 -> N-0000016
- U1 pad 11: N-0000014 -> N-0000015
- U1 pad 12: N-000002 -> N-000005
- U1 pad 2: N-0000020 -> N-0000024
- U1 pad 3: N-0000012 -> N-0000022
- U1 pad 4: N-0000017 -> N-0000021
- U1 pad 5: N-0000010 -> N-000004
- U1 pad 6: N-000009 -> N-000003
- U1 pad 7: N-0000019 -> N-0000017
- U1 pad 8: N-0000011 -> N-0000018
- U1 pad 9: N-0000016 -> N-0000014
Routing:
- net /GND: track 0.00 -> 28.4 mm, vias 0 -> 12
- net /fixation_target_module_6/GND: track 157.7 -> 131.4 mm
- net N-0000015: track 44.1 -> 25.7 mm, vias 10 -> 5
- net N-000002: track 7.18 -> 25.7 mm, vias 0 -> 5
- net /V_IN: track 0.00 -> 11.2 mm, vias 0 -> 6
- net N-0000022: track 0.00 -> 10.9 mm
- net N-0000012: track 21.8 -> 10.9 mm
- net N-0000019: track 20.0 -> 10.0 mm
- net N-000009: track 17.3 -> 8.67 mm
- net N-000003: track 0.00 -> 8.67 mm
- net N-0000014: track 7.18 -> 15.8 mm
- net N-0000016: track 24.4 -> 15.8 mm
- net N-0000017: track 4.01 -> 12.0 mm
- net N-0000023: track 0.00 -> 7.36 mm
- net N-0000011: track 12.7 -> 6.34 mm
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- added copper zone on B.Cu, net /GND
- added copper zone on F.Cu, net /GND
- added copper zone on B.Cu, net /V_IN
- added copper zone on F.Cu, net /V_IN
Other:
- net class 20mil added: clearance 0.254, trace_width 0.508, via_dia 0.762, via_drill 0.381
