File: kicad/spiky_sphere_reborn.kicad_pcb (KiCad board)
At the start: 2 copper layers, 0 parts

Commit message: working on new masks
Parts:
- added 1PIN: P***, 1pin, F.Cu at (183.0, 134.0)
- added 1PIN: P***, 1pin, F.Cu at (196.0, 122.8)
- added 1PIN: P***, 1pin, F.Cu at (208.7, 122.8)
- added 1PIN: P***, 1pin, F.Cu at (170.6, 122.8)
- added 1PIN: P***, 1pin, F.Cu at (170.6, 110.1)
- added 1PIN: P***, 1pin, F.Cu at (183.3, 110.1)
- added 1PIN: P***, 1pin, F.Cu at (196.0, 110.1)
- added 1PIN: P***, 1pin, F.Cu at (208.7, 110.1)
